File: Low-freq-Amplifer-offset/LFAmp-offset.kicad_pcb (KiCad board)
At the start: 2 copper layers, 35 parts, among them J1 Conn_01x03_Pin, J2 Conn_Coaxial, J3 Conn_Coaxial, U1 OPA1602, U2 LM317_SOT-223, U3 LM337_SOT223

Commit message: BOM and Board are added
Parts:
- added REF**: MountingHole_2.2mm_M2, MountingHole:MountingHole_2.2mm_M2, F.Cu at (211.0, 106.0)
- added REF**: MountingHole_2.2mm_M2, MountingHole:MountingHole_2.2mm_M2, F.Cu at (211.0, 63.0)
- added REF**: MountingHole_2.2mm_M2, MountingHole:MountingHole_2.2mm_M2, F.Cu at (168.0, 106.0)
- added REF**: MountingHole_2.2mm_M2, MountingHole:MountingHole_2.2mm_M2, F.Cu at (168.0, 63.0)
- C8: moved to B.Cu
- moved J3 185.0 mm to (197.5, 106.5), turned to -90 degrees
- moved R8 178.5 mm to (204.0, 93.5), turned to -90 degrees
- moved J2 174.8 mm to (197.0, 63.4), turned to 90 degrees
- moved R9 174.0 mm to (201.0, 90.0), turned to 90 degrees
- moved R5 172.6 mm to (197.5, 71.0), turned to -90 degrees
- moved R3 170.1 mm to (186.0, 105.5), turned to 90 degrees
- moved R4 169.9 mm to (188.5, 100.5), turned to 90 degrees
- moved R11 169.6 mm to (197.5, 96.5), turned to -90 degrees
- moved R7 168.1 mm to (195.0, 83.5), turned to -90 degrees
- moved R2 161.6 mm to (186.0, 65.0), turned to 180 degrees
- moved R6 159.7 mm to (186.0, 81.5), turned to -90 degrees
- moved C9 159.2 mm to (197.0, 91.5), turned to -90 degrees
- moved R1 157.8 mm to (181.5, 66.5), turned to -90 degrees
- moved R13 154.8 mm to (189.0, 77.0)
- moved R12 154.6 mm to (178.5, 107.5)
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Connections:
- D3 pad 1: Net-(D3-K) -> GND
- D3 pad 2: +5V -> Net-(D3-A)
- J3 pad 1: GND -> Net-(J3-In)
- J3 pad 2: Net-(J3-Ext) -> GND
- R11 pad 2: Net-(J3-Ext) -> Net-(J3-In)
- R12 pad 1: Net-(D3-K) -> +5V
- R12 pad 2: GND -> Net-(D3-A)
Routing:
- net +5V: track 0.00 -> 93.1 mm, vias 0 -> 3
- net -5V: track 0.00 -> 51.8 mm, vias 0 -> 2
- net Net-(U1B--): track 0.00 -> 34.6 mm, vias 0 -> 2
- net Net-(C10-Pad2): track 0.00 -> 33.4 mm
- net Net-(U1A--): track 0.00 -> 25.9 mm
- net Net-(C9-Pad2): track 0.00 -> 22.5 mm
- net Net-(U3-ADJ): track 0.00 -> 15.9 mm
- net Net-(U2-ADJ): track 0.00 -> 14.4 mm
- net Net-(R10-Pad2): track 0.00 -> 11.6 mm
- net Net-(J3-In): track 0.00 -> 9.71 mm
- net Net-(D1-A): track 0.00 -> 9.36 mm
- net Net-(D4-A): track 0.00 -> 9.20 mm, vias 0 -> 2
- net Net-(D2-K): track 0.00 -> 8.74 mm
- net -15V: track 0.00 -> 8.25 mm
- net Net-(J2-In): track 0.00 -> 6.42 mm
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- added copper zone on B.Cu, net GND
- added copper zone on F.Cu, net GND
Other:
- board outline added: 50 x 50 mm
- board text added: "+15V"
- board text added: "-15V"
- board text added: "GND"
- board text added: "Gain"
- board text added: "IN"
- board text added: "OUT"
- board text added: "Offset"
