File: Low-freq-Amplifer-offset/LFAmp-offset.kicad_sch (KiCad schematic)
At the start: 29 parts, among them J1 Conn_01x03_Pin, J2 Conn_Coaxial, J3 Conn_Coaxial, U1 OPA1602, U2 LM317_SOT-223, U3 LM337_SOT223

Commit message: bom
Parts:
- added D1, D2: D, Diode_SMD:D_1206_3216Metric, symbol Device:D
- added D3, D4: LED, Diode_SMD:D_1206_3216Metric, symbol Device:LED
- added R12, R13: 50kR, Resistor_SMD:R_1206_3216Metric, symbol Device:R
- R11: value 0R -> 50R
Connections:
- net +15V: now also D1.1 (K); no longer C1.1, J1.3 (Pin_3)
- net +5V: now also D3.2 (A)
- net -15V: now also D2.2 (A); no longer C2.1, J1.1 (Pin_1)
- net -5V: now also D4.1 (K)
- net GND: now also R12.2, R13.2
- new net: C1.1, D1.2 (A), J1.3 (Pin_3)
- new net: D4.2 (A), R13.1
- new net: D3.1 (K), R12.1
- new net: C2.1, D2.1 (K), J1.1 (Pin_1)
Other:
- moved on the sheet: C1, C2, J1

Commit message: BOM and Board are added
Connections:
- net +5V: now also R12.1; no longer D3.2 (A)
- net GND: now also D3.1 (K), J3.2 (Ext); no longer J3.1 (In), R12.2
- net at R11.2: now also J3.1 (In); no longer J3.2 (Ext)
- new net: D3.2 (A), R12.2
Other:
- moved on the sheet: D3, J3, R12
Changed lines of the file:
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@@
 	(wire
 		(pts
+			(xy 180.34 97.79) (xy 171.45 97.79)
+		)
+		(stroke
+			(width 0)
+			(type default)
+		)
+	)
+	(wire
+		(pts
 			(xy 66.04 31.75) (xy 66.04 34.29)
 		)
@@
 	(wire
 		(pts
+			(xy 171.45 97.79) (xy 171.45 96.52)
+		)
+		(stroke
+			(width 0)
+			(type default)
+		)
+	)
+	(wire
+		(pts
 			(xy 92.71 24.13) (xy 92.71 27.94)
 		)
@@
 	(wire
 		(pts
-			(xy 172.72 91.44) (xy 176.53 91.44)
+			(xy 185.42 106.68) (xy 185.42 102.87)
 		)
 		(stroke
@@
 	(symbol
 		(lib_id "power:GND")
-		(at 172.72 91.44 270)
+		(at 185.42 106.68 0)
 		(unit 1)
 		(exclude_from_sim no)
@@
 		(fields_autoplaced yes)
 		(property "Reference" "#PWR025"
-			(at 166.37 91.44 0)
+			(at 185.42 113.03 0)
 			(effects
 				(font
@@
 		)
 		(property "Value" "GND"
-			(at 168.91 91.4399 90)
+			(at 185.4199 110.49 90)
 			(effects
 				(font
@@
 		)
 		(property "Footprint" ""
-			(at 172.72 91.44 0)
+			(at 185.42 106.68 0)
 			(effects
 				(font
@@
 		)
 		(property "Datasheet" ""
-			(at 172.72 91.44 0)
+			(at 185.42 106.68 0)
 			(effects
 				(font
@@
 		)
 		(property "Description" "Power symbol creates a global label with name \"GND\" , ground"
-			(at 172.72 91.44 0)
+			(at 185.42 106.68 0)
 			(effects
 				(font
@@
 			)
 		)
+		(property "Sim.Library" "/home/evgeny/Downloads/OPA1602.lib"
+			(at 111.76 54.61 0)
+			(effects
+				(font
+					(size 1.27 1.27)
+				)
+				(hide yes)
+			)
+		)
+		(property "Sim.Name" "OPA1602"
+			(at 111.76 54.61 0)
+			(effects
+				(font
+					(size 1.27 1.27)
+				)
+				(hide yes)
+			)
+		)
+		(property "Sim.Device" "SUBCKT"
+			(at 111.76 54.61 0)
+			(effects
+				(font
+					(size 1.27 1.27)
+				)
+				(hide yes)
+			)
+		)
+		(property "Sim.Pins" "4=V- 5=+IN 6=-IN 7=Vout 8=V+"
+			(at 111.76 54.61 0)
+			(effects
+				(font
+					(size 1.27 1.27)
+				)
+				(hide yes)
+			)
+		)
 		(pin "7"
 		)
@@
 	(symbol
 		(lib_id "Connector:Conn_Coaxial")
-		(at 176.53 96.52 270)
+		(at 185.42 97.79 0)
 		(unit 1)
 		(exclude_from_sim no)
@@
 		(fields_autoplaced yes)
 		(property "Reference" "J3"
-			(at 180.34 94.9324 90)
+			(at 189.23 96.8131 0)
 			(effects
 				(font
@@
 		)
 		(property "Value" "Conn_Coaxial"
-			(at 180.34 97.4724 90)
+			(at 189.23 99.3531 0)
 			(effects
 				(font
@@
 		)
 		(property "Footprint" "Connector_Coaxial:SMA_Amphenol_132289_EdgeMount"
-			(at 176.53 96.52 0)
+			(at 185.42 97.79 0)
 			(effects
 				(font
@@
 		)
 		(property "Datasheet" "~"
-			(at 176.53 96.52 0)
+			(at 185.42 97.79 0)
 			(effects
 				(font
@@
 		)
 		(property "Description" "coaxial connector (BNC, SMA, SMB, SMC, Cinch/RCA, LEMO, ...)"
-			(at 176.53 96.52 0)
+			(at 185.42 97.79 0)
 			(effects
 				(font
@@
 	(symbol
 		(lib_id "Device:LED")
-		(at 92.71 31.75 90)
+		(at 92.71 39.37 90)
 		(unit 1)
 		(exclude_from_sim no)
@@
 		(fields_autoplaced yes)
 		(property "Reference" "D3"
-			(at 96.52 32.0674 90)
+			(at 96.52 39.6874 90)
 			(effects
 				(font
@@
 		)
 		(property "Value" "LED"
-			(at 96.52 34.6074 90)
+			(at 96.52 42.2274 90)
 			(effects
 				(font
@@
 		)
 		(property "Footprint" "Diode_SMD:D_1206_3216Metric"
-			(at 92.71 31.75 0)
+			(at 92.71 39.37 0)
 			(effects
 				(font
@@
 		)
 		(property "Datasheet" "~"
-			(at 92.71 31.75 0)
+			(at 92.71 39.37 0)
 			(effects
 				(font
@@
 		)
 		(property "Description" "Light emitting diode"
-			(at 92.71 31.75 0)
+			(at 92.71 39.37 0)
 			(effects
 				(font
@@
 		)
 		(property "Sim.Pins" "1=K 2=A"
-			(at 92.71 31.75 0)
+			(at 92.71 39.37 0)
 			(effects
 				(font
@@
 		)
 		(instances
-			(project ""
+			(project "LFAmp-offset"
 				(path "/393cb05a-92c1-4d36-8b2e-3dda6e9e550e"
 					(reference "D3")
@@
 			)
 		)
+		(property "Sim.Library" "/home/evgeny/Downloads/OPA1602.lib"
+			(at 146.05 96.52 0)
+			(effects
+				(font
+					(size 1.27 1.27)
+				)
+				(hide yes)
+			)
+		)
+		(property "Sim.Name" "OPA1602"
+			(at 146.05 96.52 0)
+			(effects
+				(font
+					(size 1.27 1.27)
+				)
+				(hide yes)
+			)
+		)
+		(property "Sim.Device" "SUBCKT"
+			(at 146.05 96.52 0)
+			(effects
+				(font
+					(size 1.27 1.27)
+				)
+				(hide yes)
+			)
+		)
+		(property "Sim.Pins" "4=V- 5=+IN 6=-IN 7=Vout 8=V+"
+			(at 146.05 96.52 0)
+			(effects
+				(font
+					(size 1.27 1.27)
+				)
+				(hide yes)
+			)
+		)
 		(pin "7"
 		)
@@
 	(symbol
 		(lib_id "Device:R")
-		(at 92.71 39.37 0)
+		(at 92.71 31.75 0)
 		(unit 1)
 		(exclude_from_sim no)
@@
 		(fields_autoplaced yes)
 		(property "Reference" "R12"
-			(at 95.25 38.0999 0)
+			(at 95.25 30.4799 0)
 			(effects
 				(font
@@
 		)
 		(property "Value" "50kR"
-			(at 95.25 40.6399 0)
+			(at 95.25 33.0199 0)
 			(effects
 				(font
@@
 		)
 		(property "Footprint" "Resistor_SMD:R_1206_3216Metric"
-			(at 90.932 39.37 90)
+			(at 90.932 31.75 90)
 			(effects
 				(font
@@
 		)
 		(property "Datasheet" "~"
-			(at 92.71 39.37 0)
+			(at 92.71 31.75 0)
 			(effects
 				(font
@@
 		)
 		(property "Description" "Resistor"
-			(at 92.71 39.37 0)
+			(at 92.71 31.75 0)
 			(effects
 				(font
@@
 			(at 85.09 99.06 0)
 			(effects
+				(font
+					(size 1.27 1.27)
+				)
+				(hide yes)
+			)
+		)
+		(property "Sim.Library" "/home/evgeny/Downloads/OPA1602.lib"
+			(at 85.09 99.06 0)
+			(effects
+				(font
+					(size 1.27 1.27)
+				)
+				(hide yes)
+			)
+		)
+		(property "Sim.Name" "OPA1602"
+			(at 85.09 99.06 0)
+			(effects
+				(font
+					(size 1.27 1.27)
+				)
+				(hide yes)
+			)
+		)
+		(property "Sim.Device" "SUBCKT"
+			(at 85.09 99.06 0)
+			(effects
+				(font
+					(size 1.27 1.27)
+				)
+				(hide yes)
+			)
+		)
+		(property "Sim.Pins" "4=V- 5=+IN 6=-IN 7=Vout 8=V+"
+			(at 85.09 99.06 0)
+			(effects
